File: mfos_vco_shapers.brd (EAGLE design)
At the start: 100 x 80 mm, 48 parts, among them IC1 TL072P, IC2 TL072P, IC3 LM13700N

Commit message: better spacing and polarized caps
Parts:
- removed R5: 10k, pot:B64Y
- added TRI_OFFSET: 10k, pot:B64Y
- C3, C4: device rcl:C050-024X044 -> rcl:B45181B
- moved TRI 53.3 mm to (78.7, 0.00)
- moved JP1 51.4 mm to (11.4, 45.7), turned to 270 degrees
- moved SINE_SHAPE 48.0 mm to (72.4, 60.1)
- moved D3 43.0 mm to (5.71, 41.3), turned to 270 degrees
- moved R16 42.4 mm to (80.8, 57.1), turned to 270 degrees
- moved D2 41.0 mm to (7.62, 34.3), turned to 90 degrees
- moved R9 39.5 mm to (47.5, 28.8), turned to 90 degrees
- moved R13 39.4 mm to (34.2, 42.8), turned to 270 degrees
- moved C2 33.0 mm to (15.2, 29.2), turned to 90 degrees
- moved R4 31.8 mm to (63.9, 23.0)
- moved D6 30.2 mm to (24.8, 24.8), turned to 180 degrees
- moved D1 29.6 mm to (24.8, 32.4)
- moved D5 28.5 mm to (24.8, 27.3), turned to 0 degrees
- moved D4 27.5 mm to (24.8, 29.8), turned to 180 degrees
- moved R6 27.5 mm to (62.2, 53.1)
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Connections:
- net GND: now also C3.-, C4.+, SIN.P$1, TRI_OFFSET.A; no longer C3.2, C4.1, R5.A
- net N$10: now also C3.+; no longer C3.1
- net N$7: now also TRI_OFFSET.E; no longer R5.E
- net N$8: now also TRI_OFFSET.S; no longer R5.S
- net N$9: now also C4.-; no longer C4.2
Routing:
- net -12V: track 43.9 -> 109.3 mm, vias 0 -> 4
- net N$10: track 83.7 -> 26.4 mm
- net N$24: track 0.00 -> 56.6 mm
- net N$11: track 44.7 -> 97.5 mm
- net +12V: track 67.8 -> 119.7 mm
- net N$20: track 10.1 -> 46.3 mm
- net N$15: track 41.4 -> 9.39 mm
- net N$5: track 15.5 -> 43.5 mm, vias 0 -> 2
- net N$3: track 46.0 -> 72.9 mm, vias 0 -> 2
- net N$17: track 36.9 -> 63.6 mm
- net N$35: track 43.2 -> 68.7 mm
- net GND: track 264.6 -> 288.2 mm, vias 0 -> 6
- net N$26: track 7.69 -> 29.3 mm
- net N$27: track 28.2 -> 8.61 mm
- net N$28: track 26.7 -> 10.4 mm
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Other:
- board size 100 x 80 mm -> 100 x 81 mm
