File: mfos_vco_shapers.brd (EAGLE design)
At the start: 100 x 80 mm, 48 parts, among them IC1 TL072P, IC2 TL072P, IC3 LM13700N

Commit message: layout tweaks
Parts:
- removed JP1: (no value), SparkFun-Connectors:1X05_LOCK_LONGPADS
- added X3: 22-23-2051, con-molex:22-23-2051
- moved R6 6.65 mm to (63.0, 50.0), turned to 0 degrees
- moved R1 5.15 mm to (56.0, 53.6), turned to 270 degrees
- moved R2 3.41 mm to (63.8, 53.7)
- moved TRI_OFFSET 3.25 mm to (50.4, 53.2)
- moved R10 2.55 mm to (38.4, 22.2)
- moved R9 2.18 mm to (41.5, 30.7)
- moved D3 1.80 mm to (3.94, 41.0)
- moved D2 1.78 mm to (5.84, 34.3)
- moved R15 0.51 mm to (19.7, 11.7)
Connections:
- net +12V: now also X3.3; no longer JP1.3
- net -12V: now also X3.1; no longer JP1.1
- net GND: now also X3.2; no longer JP1.2
- net N$33: now also X3.4; no longer JP1.4
- net N$35: now also X3.5; no longer JP1.5
Routing:
- net N$13: track 55.1 -> 72.1 mm
- net N$3: track 73.1 -> 83.4 mm
- net N$7: track 13.5 -> 19.6 mm
- net N$11: track 98.3 -> 93.9 mm
- net N$35: track 63.5 -> 61.4 mm
- net N$8: track 20.9 -> 18.9 mm
- net N$15: track 10.3 -> 12.0 mm
- net +12V: track 122.4 -> 124.0 mm
- net N$5: track 88.3 -> 86.8 mm
- net N$10: track 26.4 -> 27.9 mm
- net N$33: track 3.56 -> 4.83 mm
- net N$4: track 7.57 -> 8.71 mm
- net N$14: track 13.0 -> 12.0 mm
- net -12V: track 107.5 -> 108.3 mm

Commit message: tweak
Parts:
- moved C4 4.57 mm to (33.7, 35.8)
- moved C7 4.57 mm to (52.2, 43.2)
- moved C9 4.57 mm to (42.4, 43.2)
- moved IC1 4.57 mm to (59.8, 43.2)
- moved IC3 4.57 mm to (77.3, 29.7)
- moved PWM 4.57 mm to (40.8, 0.00)
- moved R1 4.57 mm to (60.6, 53.6)
- moved R10 4.57 mm to (42.9, 22.2)
- moved R12 4.57 mm to (58.7, 27.2)
- moved R13 4.57 mm to (38.7, 42.5)
- moved R14 4.57 mm to (50.3, 20.3)
- moved R15 4.57 mm to (24.3, 11.7)
- moved R16 4.57 mm to (86.4, 53.8)
- moved R19 4.57 mm to (88.1, 25.1)
- moved R20 4.57 mm to (88.1, 36.1)
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Routing:
- net N$11: track 93.9 -> 94.6 mm
