File: mfos_vco_shapers.sch (EAGLE design)
At the start: 48 parts, among them IC1 TL072P, IC2 TL072P, IC3 LM13700N

Commit message: better spacing and polarized caps
Parts:
- C3, C4: device rcl:C-US050-024X044 -> rcl:CPOL-USB45181B
- renumbered R5 to TRI_OFFSET
Connections:
- net GND: now also C3.-, C4.+, SIN.RING; no longer C3.2, C4.1
- net N$10: now also C3.+; no longer C3.1
- net N$9: now also C4.-; no longer C4.2
Other:
- moved on the sheet: SIN
Changed lines of the file:
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@@
 <grid distance="0.1" unitdist="inch" unit="inch" style="lines" multiple="1" display="no" altdistance="0.01" altunitdist="inch" altunit="inch"/>
 <layers>
-<layer number="1" name="Top" color="4" fill="1" visible="no" active="no"/>
-<layer number="16" name="Bottom" color="1" fill="1" visible="no" active="no"/>
-<layer number="17" name="Pads" color="2" fill="1" visible="no" active="no"/>
-<layer number="18" name="Vias" color="2" fill="1" visible="no" active="no"/>
-<layer number="19" name="Unrouted" color="6" fill="1" visible="no" active="no"/>
-<layer number="20" name="Dimension" color="15" fill="1" visible="no" active="no"/>
-<layer number="21" name="tPlace" color="7" fill="1" visible="no" active="no"/>
-<layer number="22" name="bPlace" color="7" fill="1" visible="no" active="no"/>
-<layer number="23" name="tOrigins" color="15" fill="1" visible="no" active="no"/>
-<layer number="24" name="bOrigins" color="15" fill="1" visible="no" active="no"/>
-<layer number="25" name="tNames" color="7" fill="1" visible="no" active="no"/>
-<layer number="26" name="bNames" color="7" fill="1" visible="no" active="no"/>
-<layer number="27" name="tValues" color="7" fill="1" visible="no" active="no"/>
-<layer number="28" name="bValues" color="7" fill="1" visible="no" active="no"/>
+<layer number="1" name="Top" color="4" fill="1" visible="yes" active="no"/>
+<layer number="16" name="Bottom" color="1" fill="1" visible="yes" active="no"/>
+<layer number="17" name="Pads" color="2" fill="1" visible="yes" active="no"/>
+<layer number="18" name="Vias" color="2" fill="1" visible="yes" active="no"/>
+<layer number="19" name="Unrouted" color="6" fill="1" visible="yes" active="no"/>
+<layer number="20" name="Dimension" color="15" fill="1" visible="yes" active="no"/>
+<layer number="21" name="tPlace" color="7" fill="1" visible="yes" active="no"/>
+<layer number="22" name="bPlace" color="7" fill="1" visible="yes" active="no"/>
+<layer number="23" name="tOrigins" color="15" fill="1" visible="yes" active="no"/>
+<layer number="24" name="bOrigins" color="15" fill="1" visible="yes" active="no"/>
+<layer number="25" name="tNames" color="7" fill="1" visible="yes" active="no"/>
+<layer number="26" name="bNames" color="7" fill="1" visible="yes" active="no"/>
+<layer number="27" name="tValues" color="7" fill="1" visible="yes" active="no"/>
+<layer number="28" name="bValues" color="7" fill="1" visible="yes" active="no"/>
 <layer number="29" name="tStop" color="7" fill="3" visible="no" active="no"/>
 <layer number="30" name="bStop" color="7" fill="6" visible="no" active="no"/>
@@
 <layer number="35" name="tGlue" color="7" fill="4" visible="no" active="no"/>
 <layer number="36" name="bGlue" color="7" fill="5" visible="no" active="no"/>
-<layer number="37" name="tTest" color="7" fill="1" visible="no" active="no"/>
-<layer number="38" name="bTest" color="7" fill="1" visible="no" active="no"/>
+<layer number="37" name="tTest" color="7" fill="1" visible="yes" active="no"/>
+<layer number="38" name="bTest" color="7" fill="1" visible="yes" active="no"/>
 <layer number="39" name="tKeepout" color="4" fill="11" visible="no" active="no"/>
 <layer number="40" name="bKeepout" color="1" fill="11" visible="no" active="no"/>
@@
 <layer number="44" name="Drills" color="7" fill="1" visible="no" active="no"/>
 <layer number="45" name="Holes" color="7" fill="1" visible="no" active="no"/>
-<layer number="46" name="Milling" color="3" fill="1" visible="no" active="no"/>
-<layer number="47" name="Measures" color="7" fill="1" visible="no" active="no"/>
-<layer number="48" name="Document" color="7" fill="1" visible="no" active="no"/>
-<layer number="49" name="Reference" color="7" fill="1" visible="no" active="no"/>
-<layer number="50" name="dxf" color="7" fill="1" visible="no" active="no"/>
-<layer number="51" name="tDocu" color="7" fill="1" visible="no" active="no"/>
-<layer number="52" name="bDocu" color="7" fill="1" visible="no" active="no"/>
-<layer number="53" name="tGND_GNDA" color="7" fill="9" visible="no" active="no"/>
-<layer number="54" name="bGND_GNDA" color="1" fill="9" visible="no" active="no"/>
-<layer number="56" name="wert" color="7" fill="1" visible="no" active="no"/>
-<layer number="57" name="tCAD" color="7" fill="1" visible="no" active="no"/>
+<layer number="46" name="Milling" color="3" fill="1" visible="yes" active="no"/>
+<layer number="47" name="Measures" color="7" fill="1" visible="yes" active="no"/>
+<layer number="48" name="Document" color="7" fill="1" visible="yes" active="no"/>
+<layer number="49" name="Reference" color="7" fill="1" visible="yes" active="no"/>
+<layer number="50" name="dxf" color="7" fill="1" visible="yes" active="no"/>
+<layer number="51" name="tDocu" color="7" fill="1" visible="yes" active="no"/>
+<layer number="52" name="bDocu" color="7" fill="1" visible="yes" active="no"/>
+<layer number="53" name="tGND_GNDA" color="7" fill="9" visible="yes" active="no"/>
+<layer number="54" name="bGND_GNDA" color="1" fill="9" visible="yes" active="no"/>
+<layer number="56" name="wert" color="7" fill="1" visible="yes" active="no"/>
+<layer number="57" name="tCAD" color="7" fill="1" visible="yes" active="no"/>
 <layer number="90" name="Modules" color="5" fill="1" visible="yes" active="yes"/>
 <layer number="91" name="Nets" color="2" fill="1" visible="yes" active="yes"/>
@@
 <part name="TRI" library="erthenvar" deviceset="AUDIO-JACK" device=""/>
 <part name="C1" library="rcl" deviceset="C-US" device="050-030X075" value="0.1uF"/>
-<part name="R5" library="pot" deviceset="TRIM_US-" device="B64Y" value="10k"/>
+<part name="TRI_OFFSET" library="pot" deviceset="TRIM_US-" device="B64Y" value="10k"/>
 <part name="R6" library="rcl" deviceset="R-US_" device="0207/7" value="10k"/>
 <part name="P+1" library="supply1" deviceset="+12V" device=""/>
@@
 <part name="C2" library="rcl" deviceset="C-US" device="050-030X075" value="0.002uF"/>
 <part name="P-1" library="supply1" deviceset="-12V" device=""/>
-<part name="C3" library="rcl" deviceset="C-US" device="050-024X044" value="1uF"/>
-<part name="C4" library="rcl" deviceset="C-US" device="050-024X044" value="1uF"/>
+<part name="C3" library="rcl" deviceset="CPOL-US" device="B45181B" value="1uF"/>
+<part name="C4" library="rcl" deviceset="CPOL-US" device="B45181B" value="1uF"/>
 <part name="GND3" library="supply1" deviceset="GND" device=""/>
 <part name="R8" library="pot" deviceset="3RP/1610N" device="" value="100k"/>
@@
 <part name="GND11" library="supply1" deviceset="GND" device=""/>
 <part name="GND12" library="supply1" deviceset="GND" device=""/>
+<part name="GND13" library="supply1" deviceset="GND" device=""/>
 </parts>
 <sheets>
@@
 <instance part="TRI" gate="G$1" x="142.24" y="93.98" rot="R180"/>
 <instance part="C1" gate="G$1" x="68.58" y="111.76"/>
-<instance part="R5" gate="G$1" x="68.58" y="124.46" rot="R270"/>
+<instance part="TRI_OFFSET" gate="G$1" x="68.58" y="124.46" rot="R270"/>
 <instance part="R6" gate="G$1" x="83.82" y="124.46"/>
 <instance part="P+1" gate="1" x="93.98" y="127"/>
@@
 <instance part="GND8" gate="1" x="170.18" y="-22.86"/>
 <instance part="R22" gate="G$1" x="170.18" y="-10.16"/>
-<instance part="SIN" gate="G$1" x="190.5" y="-5.08" rot="R180"/>
+<instance part="SIN" gate="G$1" x="193.04" y="-5.08" rot="R180"/>
 <instance part="R23" gate="G$1" x="175.26" y="0"/>
 <instance part="P-4" gate="1" x="180.34" y="-17.78"/>
@@
 <instance part="GND11" gate="1" x="149.86" y="71.12"/>
 <instance part="GND12" gate="1" x="233.68" y="55.88"/>
+<instance part="GND13" gate="1" x="185.42" y="-10.16"/>
 </instances>
 <busses>
@@
 </segment>
 <segment>
-<pinref part="R5" gate="G$1" pin="A"/>
+<pinref part="TRI_OFFSET" gate="G$1" pin="A"/>
 <pinref part="GND1" gate="1" pin="GND"/>
 <wire x1="58.42" y1="124.46" x2="60.96" y2="124.46" width="0.1524" layer="91"/>
@@
 <pinref part="GND3" gate="1" pin="GND"/>
 <wire x1="139.7" y1="27.94" x2="139.7" y2="30.48" width="0.1524" layer="91"/>
-<pinref part="C4" gate="G$1" pin="1"/>
+<pinref part="C4" gate="G$1" pin="+"/>
 <wire x1="139.7" y1="30.48" x2="127" y2="30.48" width="0.1524" layer="91"/>
-<pinref part="C3" gate="G$1" pin="2"/>
+<pinref part="C3" gate="G$1" pin="-"/>
 <wire x1="127" y1="43.18" x2="139.7" y2="43.18" width="0.1524" layer="91"/>
 <wire x1="139.7" y1="43.18" x2="139.7" y2="30.48" width="0.1524" layer="91"/>
@@
 <pinref part="SQR" gate="G$1" pin="RING"/>
 <pinref part="GND12" gate="1" pin="GND"/>
+</segment>
+<segment>
+<pinref part="SIN" gate="G$1" pin="RING"/>
+<pinref part="GND13" gate="1" pin="GND"/>
 </segment>
 </net>
@@
 <net name="N$7" class="0">
 <segment>
-<pinref part="R5" gate="G$1" pin="E"/>
+<pinref part="TRI_OFFSET" gate="G$1" pin="E"/>
 <pinref part="R6" gate="G$1" pin="1"/>
 <wire x1="78.74" y1="124.46" x2="76.2" y2="124.46" width="0.1524" layer="91"/>
@@
 <wire x1="99.06" y1="101.6" x2="76.2" y2="101.6" width="0.1524" layer="91"/>
 <wire x1="76.2" y1="101.6" x2="76.2" y2="116.84" width="0.1524" layer="91"/>
-<pinref part="R5" gate="G$1" pin="S"/>
+<pinref part="TRI_OFFSET" gate="G$1" pin="S"/>
 <pinref part="C1" gate="G$1" pin="1"/>
 <wire x1="68.58" y1="114.3" x2="68.58" y2="116.84" width="0.1524" layer="91"/>
@@
 <net name="N$9" class="0">
 <segment>
-<pinref part="C4" gate="G$1" pin="2"/>
+<pinref part="C4" gate="G$1" pin="-"/>
 <pinref part="D6" gate="G$1" pin="A"/>
 <wire x1="119.38" y1="30.48" x2="114.3" y2="30.48" width="0.1524" layer="91"/>
@@
 <net name="N$10" class="0">
 <segment>
-<pinref part="C3" gate="G$1" pin="1"/>
+<pinref part="C3" gate="G$1" pin="+"/>
 <pinref part="D3" gate="G$1" pin="C"/>
 <wire x1="119.38" y1="43.18" x2="114.3" y2="43.18" width="0.1524" layer="91"/>
@@
 <pinref part="SIN" gate="G$1" pin="TIP"/>
 <pinref part="R23" gate="G$1" pin="2"/>
-<wire x1="180.34" y1="0" x2="182.88" y2="0" width="0.1524" layer="91"/>
-</segment>
-</net>
+<wire x1="180.34" y1="0" x2="185.42" y2="0" width="0.1524" layer="91"/>
+</segment>
+</net>

Commit message: layout tweaks
Parts:
- removed JP1: (no value), SparkFun-Connectors:M05LOCK_LONGPADS
- added X3: 22-23-2051, con-molex:22-23-2051
Connections:
- net +12V: now also X3-3.S; no longer JP1.3
- net -12V: now also X3-1.S; no longer JP1.1
- net GND: now also X3-2.S; no longer JP1.2
- net N$33: now also X3-4.S; no longer JP1.4
- net N$35: now also X3-5.S; no longer JP1.5
